File: MSX_VDP_Tester_Arduino/MSX_VDP_Tester_Arduino.kicad_sch (KiCad schematic)
At the start: 22 parts, among them J1 VDP Under Test, J2 +5V In, J3 Power Passthrough, SW1 Test, U1 74LS595, U2 HDSP-7803, Y1 21.47MHz

Commit message: Initial version for testing
Parts:
- J1: footprint Package_DIP:DIP-64_W15.24mm_Socket_LongPads -> Clueless_Engineer:DIPS1905W50P178L5730H420Q64N
Changed lines of the file:
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@@
 	(title_block
 		(title "MSX VDP Tester")
-		(date "3/JUL/2026")
-		(rev "WIP")
+		(date "5/JUL/2026")
+		(rev "A")
 		(company "Brett Hallen")
 	)
@@
 			)
 		)
-		(property "Footprint" "Package_DIP:DIP-64_W15.24mm_Socket_LongPads"
+		(property "Footprint" "Clueless_Engineer:DIPS1905W50P178L5730H420Q64N"
 			(at 60.96 132.08 0)
 			(hide yes)
