File: MSX_VDP_Tester_Arduino/MSX_VDP_Tester_Arduino.kicad_pcb (KiCad board)
At the start: 2 copper layers, 83.8 x 61 mm, 22 parts, among them J1 VDP Under Test, J2 +5V In, J3 Power Passthrough, SW1 Test, U1 74LS595, U2 HDSP-7803, Y1 21.47MHz

Commit message: Initial version for testing
Parts:
- J1: footprint Package_DIP:DIP-64_W15.24mm_Socket_LongPads -> Clueless_Engineer:DIPS1905W50P178L5730H420Q64N
- moved C4 27.3 mm to (100.3, 134.0), turned to -90 degrees
- moved J1 24.4 mm to (114.4, 137.2)
- moved C1 21.3 mm to (110.5, 137.2)
- moved SW1 18.6 mm to (93.8, 103.8)
- moved J3 17.3 mm to (97.0, 97.0)
- moved C5 13.9 mm to (100.3, 118.7), turned to 90 degrees
- moved Y1 12.4 mm to (100.3, 123.8), turned to -90 degrees
- moved J2 8.66 mm to (97.0, 90.0), turned to -90 degrees
- moved C2 8.64 mm to (110.5, 118.1)
- moved R1 0.63 mm to (153.0, 126.4)
Routing:
- net /+5V: track 156.9 -> 204.8 mm
- net /GND: track 178.2 -> 225.2 mm
- net Net-(A1-D10): track 52.8 -> 71.8 mm
- net Net-(A1-VIN): track 14.6 -> 32.0 mm
- net /~{RESET}: track 62.9 -> 48.5 mm
- net /XTAL1: track 15.3 -> 28.1 mm
- net /XTAL2: track 14.1 -> 23.5 mm
- net /MODE1: track 39.7 -> 47.2 mm
- net /CD0: track 12.2 -> 19.3 mm
- net /MODE0: track 39.7 -> 46.5 mm
- net /CD1: track 12.9 -> 19.1 mm
- net /~{CSW}: track 39.7 -> 45.6 mm
- net /CD2: track 13.6 -> 18.0 mm
- net /CD7: track 27.1 -> 31.2 mm
- net /~{CSR}: track 39.7 -> 43.5 mm
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Other:
- board size 83.8 x 61 mm -> 84 x 64 mm
- board text added: "Brett Hallen, Jul 2026"
- board text added: "Yamaha V99x8 VDP Tester"

Commit message: Minor PCB change
Parts:
- moved C4 7.20 mm to (95.2, 128.9), turned to 180 degrees
- moved C5 7.18 mm to (95.2, 123.8), turned to 180 degrees
- moved Y1 1.27 mm to (101.6, 123.8)
Routing:
- net /GND: track 225.2 -> 236.5 mm
- net /XTAL1: track 28.1 -> 25.9 mm
- net /XTAL2: track 23.5 -> 22.7 mm
Changed lines of the file:
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@@
 	(footprint "Capacitor_THT:C_Disc_D3.0mm_W1.6mm_P2.50mm"
 		(layer "F.Cu")
-		(at 100.33 133.985 -90)
+		(at 95.23 128.905 180)
 		(descr "C, Disc series, Radial, pin pitch=2.50mm, diameter*width=3.0*1.6mm^2, Capacitor, http://www.vishay.com/docs/45233/krseries.pdf")
 		(tags "C Disc series Radial pin pitch 2.50mm diameter 3.0mm width 1.6mm Capacitor")
 		(property "Reference" "C4"
-			(at 1.25 -2.05 90)
+			(at 1.25 -2.05 0)
 			(layer "F.SilkS")
 			(hide yes)
@@
 		)
 		(property "Value" "33pF"
-			(at 1.27 3.33 0)
+			(at 1.27 -2.54 180)
 			(layer "F.SilkS")
 			(effects
@@
 		)
 		(property "Datasheet" ""
-			(at 0 0 90)
+			(at 0 0 0)
 			(layer "F.Fab")
 			(hide yes)
@@
 		)
 		(property "Description" "Unpolarized capacitor"
-			(at 0 0 90)
+			(at 0 0 0)
 			(layer "F.Fab")
 			(hide yes)
@@
 		)
 		(property "KiLib_Generator" "capacitor/THT/other"
-			(at 0 0 90)
+			(at 0 0 0)
 			(layer "F.SilkS")
 			(hide yes)
@@
 		)
 		(fp_text user "${REFERENCE}"
-			(at 1.25 0 90)
-			(layer "F.SilkS")
+			(at 1.25 0 0)
+			(layer "F.Fab")
 			(effects
 				(font
@@
 		)
 		(pad "1" thru_hole circle
-			(at 0 0 270)
+			(at 0 0 180)
 			(size 1.6 1.6)
 			(drill 0.8)
@@
 		)
 		(pad "2" thru_hole circle
-			(at 2.5 0 270)
+			(at 2.5 0 180)
 			(size 1.6 1.6)
 			(drill 0.8)
@@
 	(footprint "Capacitor_THT:C_Disc_D3.0mm_W1.6mm_P2.50mm"
 		(layer "F.Cu")
-		(at 100.33 118.745 90)
+		(at 95.25 123.825 180)
 		(descr "C, Disc series, Radial, pin pitch=2.50mm, diameter*width=3.0*1.6mm^2, Capacitor, http://www.vishay.com/docs/45233/krseries.pdf")
 		(tags "C Disc series Radial pin pitch 2.50mm diameter 3.0mm width 1.6mm Capacitor")
 		(property "Reference" "C5"
-			(at 1.25 -2.05 90)
+			(at 1.25 -2.05 0)
 			(layer "F.SilkS")
 			(hide yes)
@@
 		)
 		(property "Value" "33pF"
-			(at 1.27 -3.81 0)
+			(at 1.27 2.54 180)
 			(layer "F.SilkS")
 			(effects
@@
 		)
 		(property "Datasheet" ""
-			(at 0 0 90)
+			(at 0 0 0)
 			(layer "F.Fab")
 			(hide yes)
@@
 		)
 		(property "Description" "Unpolarized capacitor"
-			(at 0 0 90)
+			(at 0 0 0)
 			(layer "F.Fab")
 			(hide yes)
@@
 		)
 		(property "KiLib_Generator" "capacitor/THT/other"
-			(at 0 0 90)
+			(at 0 0 0)
 			(layer "F.SilkS")
 			(hide yes)
@@
 		(duplicate_pad_numbers_are_jumpers no)
 		(fp_line
-			(start 0.485 -0.92)
-			(end 2.015 -0.92)
+			(start 2.015 0.92)
+			(end 0.485 0.92)
 			(stroke
 				(width 0.12)
@@
 		)
 		(fp_line
-			(start 2.015 0.92)
-			(end 0.485 0.92)
+			(start 0.485 -0.92)
+			(end 2.015 -0.92)
 			(stroke
 				(width 0.12)
@@
 		)
 		(fp_text user "${REFERENCE}"
-			(at 1.25 0 90)
-			(layer "F.SilkS")
+			(at 1.25 0 0)
+			(layer "F.Fab")
 			(effects
 				(font
@@
 		)
 		(pad "1" thru_hole circle
-			(at 0 0 90)
+			(at 0 0 180)
 			(size 1.6 1.6)
 			(drill 0.8)
@@
 		)
 		(pad "2" thru_hole circle
-			(at 2.5 0 90)
+			(at 2.5 0 180)
 			(size 1.6 1.6)
 			(drill 0.8)
@@
 	(footprint "Crystal:Crystal_HC49-U_Vertical"
 		(layer "F.Cu")
-		(at 100.33 123.825 -90)
+		(at 101.6 123.825 -90)
 		(descr "HC-49/U, Crystal, http://5hertz.com/pdfs/04404_D.pdf")
 		(property "Reference" "Y1"
@@
 		)
 		(property "Value" "21.47MHz"
-			(at 2.54 7.33 180)
+			(at 9.525 0 180)
 			(layer "F.SilkS")
 			(effects
@@
 	)
 	(segment
-		(start 110.055 128.705)
-		(end 116.205 122.555)
+		(start 106.353485 128.705)
+		(end 116.205 118.853485)
 		(width 0.2)
 		(layer "F.Cu")
@@
 	)
 	(segment
-		(start 100.33 128.705)
-		(end 110.055 128.705)
+		(start 101.6 128.705)
+		(end 106.353485 128.705)
 		(width 0.2)
 		(layer "F.Cu")
@@
 	)
 	(segment
-		(start 116.205 122.555)
+		(start 116.205 118.853485)
 		(end 116.205 118.11)
 		(width 0.2)
@@
 	)
 	(segment
-		(start 100.33 128.705)
-		(end 100.33 133.985)
+		(start 95.23 128.905)
+		(end 101.4 128.905)
+		(width 0.2)
+		(layer "F.Cu")
+		(net "/XTAL1")
+	)
+	(segment
+		(start 101.4 128.905)
+		(end 101.6 128.705)
 		(width 0.2)
 		(layer "F.Cu")
@@
 	)
 	(segment
-		(start 100.33 136.485)
-		(end 108.665 136.485)
+		(start 92.3 106.8)
+		(end 93.75 108.25)
 		(width 0.2)
 		(layer "B.Cu")
@@
 	)
 	(segment
-		(start 92.3 106.8)
-		(end 93.75 108.25)
+		(start 121.75 85.555)
+		(end 125.73 89.535)
 		(width 0.2)
 		(layer "B.Cu")
@@
 	)
 	(segment
-		(start 121.75 85.555)
-		(end 125.73 89.535)
+		(start 110.49 134.66)
+		(end 111.927 134.66)
 		(width 0.2)
 		(layer "B.Cu")
@@
 	)
 	(segment
-		(start 106.125 116.245)
-		(end 110.49 120.61)
+		(start 93.75 108.25)
+		(end 92.75 109.25)
 		(width 0.2)
 		(layer "B.Cu")
@@
 	)
 	(segment
-		(start 110.49 134.66)
-		(end 111.927 134.66)
+		(start 92.75 129.3476)
+		(end 92.4052 129.6924)
 		(width 0.2)
 		(layer "B.Cu")
@@
 	)
 	(segment
-		(start 100.25 116.165)
-		(end 100.33 116.245)
-		(width 0.2)
-		(layer "B.Cu")
-		(net "/GND")
-	)
-	(segment
-		(start 100.33 116.245)
-		(end 106.125 116.245)
+		(start 146.05 86.32)
+		(end 144.82 86.32)
 		(width 0.2)
 		(layer "B.Cu")
@@
 	)
 	(segment
-		(start 146.05 86.32)
-		(end 144.82 86.32)
+		(start 133.35 97.155)
+		(end 133.985 97.155)
 		(width 0.2)
 		(layer "B.Cu")
@@
 	)
 	(segment
-		(start 133.35 97.155)
-		(end 133.985 97.155)
+		(start 92.75 109.25)
+		(end 92.75 123.825)
 		(width 0.2)
 		(layer "B.Cu")
@@
 	)
 	(segment
-		(start 100.25 108.25)
-		(end 100.25 116.165)
+		(start 92.73 128.905)
+		(end 98.485 134.66)
 		(width 0.2)
 		(layer "B.Cu")
@@
 	)
 	(segment
-		(start 108.665 136.485)
-		(end 110.49 134.66)
+		(start 120.65 79.375)
+		(end 121.75 80.475)
 		(width 0.2)
 		(layer "B.Cu")
@@
 	)
 	(segment
-		(start 120.65 79.375)
-		(end 121.75 80.475)
+		(start 110.49 120.61)
+		(end 110.49 134.66)
 		(width 0.2)
 		(layer "B.Cu")
@@
 	)
 	(segment
-		(start 110.49 120.61)
+		(start 98.485 134.66)
 		(end 110.49 134.66)
 		(width 0.2)
@@
 	)
 	(segment
+		(start 92.75 123.825)
+		(end 92.75 129.3476)
+		(width 0.2)
+		(layer "B.Cu")
+		(net "/GND")
+	)
+	(segment
 		(start 99.89 81.11)
 		(end 118.915 81.11)
@@
 	)
 	(segment
-		(start 100.33 123.825)
-		(end 112.0902 123.825)
+		(start 110.6678 123.825)
+		(end 114.427 120.0658)
 		(width 0.2)
 		(layer "F.Cu")
@@
 	)
 	(segment
-		(start 112.0902 123.825)
-		(end 114.427 121.4882)
+		(start 101.6 123.825)
+		(end 110.6678 123.825)
 		(width 0.2)
 		(layer "F.Cu")
@@
 	)
 	(segment
-		(start 100.33 118.745)
-		(end 100.33 123.825)
+		(start 114.427 120.0658)
+		(end 114.427 118.11)
 		(width 0.2)
 		(layer "F.Cu")
@@
 	)
 	(segment
-		(start 114.427 121.4882)
-		(end 114.427 118.11)
+		(start 95.25 123.825)
+		(end 101.6 123.825)
 		(width 0.2)
 		(layer "F.Cu")
